File: PLC/V4_final_KiCad_PCB/OP.kicad_pcb (KiCad board)
At the start: 2 copper layers, 208 x 80 mm, 304 parts, among them J1 MSTBVA-2.5-10-5.08, J10 Conn_01x03_Female, J11 Conn_01x02_Female, J12 Conn_01x15_Female, J13 01x03_fem, J14 Conn_01x15_Female, J15 01x04, J16 MSTBVA-2.5-10-5.08, J17 MSTBVA-2.5-10-5.08, J2 MSTBVA-2.5-10-5.08, J25 Conn_01x05_Female, J27 Lötauge, J28 GND_CAN opt an J33, J3 PFS 2x4, J33 opt. GND_XXX, J37 Lötauge, J4 01x08, J40 Extention, J41 Lötauge, J42 Lötauge, J43 Flachstecker, J44 Lötauge, J45 Lötauge, J46 Lötauge, J47 Lötauge, J48 Lötauge, J5 Conn_01x04, J51 Lötauge, J52 Lötauge, J6 DIN-5, J61 Lötauge, J62 Lötauge, J7 DIN-5, J8 Conn_02x02_Female, J9 Ub 0V PE, P1 1,0K lin, P2 1,0K lin, Q1 IRLML 2244, SW1 SW_DIP_x02, SW2 SW_DIP_x02, SW3 SW_DIP_x02, U1 LTV-844, U10 ADM2483xRW, U2 LTV-844, U3 LTV-844, U36 MCP3204, U39 ADuM1401xRW, U4 LTV-844, U40 ADM-803R, U42 LM4040 AIM3-2.5, U43 LM4040 AIM3-2.5, U47 ADM-809Z, U48 ADM-803L, U49 74AHC1G32, U5 MCP23S17, U50 NE555DRG4, U6 ISO1050, U7 Teensy4.0, U8 ISO1050, U9 25LC512

Commit message: V2.6 M37 PFS
Parts:
- added C95: 10u 10V, Capacitors_Tantalum_SMD:CP_Tantalum_Case-A_EIA-3216-18_Reflow, B.Cu at (163.0, 68.6)
- added R169: 10, Resistors_SMD:R_0603, F.Cu at (166.1, 76.9)
- added R171: 10, Resistors_SMD:R_0603, F.Cu at (162.8, 54.9)
- C51: value 100n -> 4µ7 16V; footprint Capacitors_SMD:C_1206_HandSoldering -> Capacitors_Tantalum_SMD:CP_Tantalum_Case-A_EIA-3216-18_Reflow
- C73, C75: footprint Capacitors_SMD:C_1206 -> Capacitors_SMD:C_0603
- D1, D10, D11, D12, D13, D14, D15, D16, D2, D3, D4, D5, D6, D7, D8, D9: value SMLVT3V3 STM -> P6SMB 5,0CA SMD
- J10: value Conn_01x03_Female -> 01x03_fem
- J11: value Conn_01x02_Female -> 01x02_fem
- J12, J14: value Conn_01x15_Female -> 01x15_fem
- J15: value 01x04 -> 01x04_fem
- J25: value Conn_01x05_Female -> 01x05_fem
- J4: value 01x08 -> 01x08_fem
- J5: value Conn_01x04 -> 01x04_fem
- J8: value Conn_02x02_Female -> 02x02_fem
- R1, R10, R11, R12, R13, R14, R15, R16, R2, R3, R4, R5, R6, R7, R8, R9: value 6k2 500mW -> 6k8 500mW
- R123, R51: value 470k -> 680k
- R133: value 47k -> 220k; moved to B.Cu
- R163, R165: footprint Capacitors_SMD:C_0603 -> Resistors_SMD:R_0603
- R17, R18, R19, R20, R21, R22, R23, R24, R25, R26, R27, R28, R29, R30, R31, R32: value 220 -> 1k1
- moved C76 5.29 mm to (162.7, 80.0), turned to 270 degrees
- moved C73 2.34 mm to (169.1, 70.9), turned to 180 degrees
- moved A2 1.73 mm to (120.7, 91.9)
- moved C1 1.14 mm to (168.8, 85.1)
- moved C75 0.90 mm to (163.0, 70.6)
- moved R133 0.55 mm to (166.2, 78.4), turned to 0 degrees
- moved U50 0.51 mm to (162.7, 74.2)
- moved C74 0.51 mm to (160.0, 79.5)
- moved C51 0.42 mm to (187.0, 43.8)
- moved C72 0.36 mm to (186.1, 57.5)
- moved U49 0.13 mm to (168.0, 68.3)
Connections:
- J4 pad 8: (no net) -> /COLDSTART_3V3INT
- R124 pad 1: Net-(Q1-Pad1) -> Net-(R124-Pad1)
- U50 pad 3: Net-(Q1-Pad1) -> Net-(R124-Pad1)
Routing:
- net /COLDSTART_3V3INT: track 0.00 -> 37.6 mm, vias 0 -> 1
- net Net-(R124-Pad1): track 0.00 -> 23.1 mm, vias 0 -> 2
- net Net-(Q1-Pad1): track 22.5 -> 0.48 mm, vias 0 -> 1
- net GNDD: track 668.1 -> 689.0 mm, vias 136 -> 152
- net Net-(U49-Pad4): track 9.39 -> 5.66 mm
- net Net-(C76-Pad1): track 11.4 -> 8.97 mm, vias 1 -> 0
- net /INTA: track 37.7 -> 39.8 mm
- net /~UART_RE: track 134.7 -> 136.2 mm
- net /INTB: track 30.8 -> 32.2 mm
- net /~RESET: track 152.8 -> 151.6 mm
- net /~SPICS_ADC: track 109.3 -> 110.3 mm
- net 5V_CPU_IN: track 117.9 -> 118.9 mm, vias 5 -> 4
- net /I_GPB0: track 40.0 -> 39.1 mm
- net /~EE_HOLD: track 104.7 -> 103.9 mm
- net /I_GPB1: track 42.0 -> 41.3 mm
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Other:
- rule trace_min: 0.2 -> 0
- board text added: "BAT 3V ~RESET ~SWMODE1 ~SWMODE2"
- board text added: "Experimental Study for PS4 1xx-MMx substitution CPU Board C.Niesen, Königswinter, Germany, CC BY-NC-SA 2023"
- board text added: "GND BUS"
- board text added: "GND_RS"
- board text added: "J3"
- board text added: "J3: BAT 3V ~RESET ~SWMODE1 ~SWMODE2"
- board text added: "J3: GNDD O O GNDD O O GNDD O O GNDD O O"
- board text added: "O O GNDD O O GNDD O O GNDD O O GNDD"
- board text added: "PFS CPU Board V2.6 M37 2023-11-23"
- board text added: "SPISCK ~SPICSIO GNDD 3V3INT 3V3EN-Q2.UP"
- board text added: "~RESET MISo MOSI SPISCK ~SPICSIO GNDD 3V3INT 3V3EN-Q2-UP"
- board text removed: "- GNDD -"
- board text removed: "Batt 3V6"
- board text removed: "Experimental Study C.Niesen, Königswinter, Germany, CC BY-NC-SA 2023"
- board text removed: "FFC CPU Board V2.6 M36 2023-07-30"
- board text removed: "GND_RS485"
- board text removed: "J3:"
- board text removed: "O"
- board text removed: "PFS CPU Board V2.6 M36 2023-07-30"
- board text removed: "SPISCK ~SPICSIO GNDD 3V3INT n.c."
- board text removed: "~Mode1"
- board text removed: "~Mode2"
- board text removed: "~RESET MISo MOSI SPISCK ~SPICSIO GNDD 3V3INT n.c."
- board text removed: "~Reset"
