File: PLC/V4_final_KiCad_PCB/UP.kicad_pcb (KiCad board)
At the start: 2 copper layers, 208 x 80 mm, 245 parts, among them J18 01x03_Male, J19 01x08_Male, J20 01x02_Male, J21 02x02_Male, J22 opt. Connector, J23 opt. Connector, J24 01x05_Male, J26 01x04, J29 Lötauge, J30 Lötauge, J31 Lötauge, J32 Lötauge, J35 Lötauge, J38 Lötauge, J39 Lötauge, J49 01x15 Male zu OP, J50 01x15 Male zu OP, J53 Lötauge, J54 Lötauge, J55 Lötauge, J56 Lötauge, J57 Lötauge, J58 Lötauge, J59 Lötauge, J60 Lötauge, J63 Lötauge, J64 Lötauge, J65 Lötauge, J66 Flachstecker, U11 2S7WA_2405_S3RP, U12 2S7WA_2405_S3RP, U13 LT1086 3.3, U14 MCP23S17, U15 LTV-844, U16 LTV-844, U17 LTV-844, U18 LTV-844, U19 BSP-452, U20 BSP-452, U21 BSP-452, U22 BSP-452, U23 BSP-452, U24 BSP-452, U25 BSP-452, U26 BSP-452, U27 BSP-452, U28 BSP-452, U29 BSP-452, U30 BSP-452, U31 BSP-452, U32 BSP-452, U33 BSP-452, U34 BSP-452, U35 ADuM1401xRW, U37 LT1086 3.3, U38 MCP4922, U41 LT 1078, U44 2S7WB_2415S3RP, U45 ADR03ARZ, U46 LCN78_05-0.5

Commit message: V2.6 M37 PFS
Parts:
- added C96: 100n, Capacitors_SMD:C_0805, B.Cu at (107.5, 76.2)
- added C97: 100n, Capacitors_SMD:C_1206, F.Cu at (104.8, 84.3)
- added J34: Brücke, mylib:Lötauge-Junction_1x1.5-0.8, F.Cu at (107.2, 73.3)
- added J36: Brücke, mylib:Lötauge-Junction_1x1.5-0.8, F.Cu at (110.0, 70.6)
- added Q2: IRLML 2244, TO_SOT_Packages_SMD:SOT-23, F.Cu at (106.4, 76.2)
- added R170: 10k, Resistors_SMD:R_0805, F.Cu at (105.9, 69.6)
- C15: moved to B.Cu
- D70, D71, D72, D73, D74, D75, D76, D77, D78, D79, D80, D81, D82, D83, D84, D85, D86, D87: value P6KE36CA -> P6KE33CA
- F4, F5: value 6A3 T -> 5,6AT
- R100, R101, R102, R103, R104, R105, R106, R107, R108, R109, R110, R111, R112, R113, R114, R115, R116, R117, R134, R135, R136, R137, R138, R139, R140, R141, R142, R143, R144, R145, R146, R147, R148, R149, R86, R87, R88, R89, R90, R91, R92, R93, R94, R95, R96, R97, R98, R99: value 6k8 -> 7k5
- moved C15 21.3 mm to (95.5, 81.5), turned to 90 degrees
- moved C82 2.22 mm to (105.7, 66.7), turned to 90 degrees
- moved C13 2.20 mm to (92.9, 80.0)
- moved C14 0.99 mm to (94.4, 85.1)
Connections:
- J19 pad 8: (no net) -> /COLDSTART_3V3INT
- U13 pad 3: /5V_CPU -> Net-(C97-Pad1)
Routing:
- net /COLDSTART_3V3INT: track 0.00 -> 145.2 mm, vias 0 -> 3
- net GNDD: track 628.4 -> 567.2 mm, vias 32 -> 46
- net +3V3: track 259.8 -> 242.4 mm
- net Net-(C97-Pad1): track 0.00 -> 8.45 mm, vias 0 -> 1
- net Net-(C13-Pad1): track 18.2 -> 20.4 mm
- net /5V_CPU: track 28.2 -> 27.4 mm, vias 3 -> 2
Other:
- board text added: "(24V)"
- board text added: "0V 24V Q0.7 Q0.6 Q0.5 Q0.4 Q0.3 Q0.2 Q0.1 Q0.0"
- board text added: "0V 24V Q1.7 Q1.6 Q1.5 Q1.4 Q1.3 Q1.2 Q1.1 Q1.0"
- board text added: "Base Board V2.6 M37 2023-11-23"
- board text added: "Br"
- board text added: "Experimental Study for PS4-1xx-MMx BaseBoard C.Niesen, Königswinter, Germany, CC BY-NC-SA 2023"
- board text added: "FFC/PFS Base Board V2.6 M37 2023-11-23"
- board text added: "GNDD"
- board text added: "PE 0V 24V"
- board text added: "Q0.0 Q0.1 Q0.2 Q0.3 Q0.4 Q0.5 Q0.6 Q0.7 24V 0V"
- board text added: "Q1.0 Q1.1 Q1.2 Q1.3 Q1.4 Q1.5 Q1.6 Q1.7 24V 0V"
- board text added: "RESET MISO MOSI SPISCK SPICSIO GNDD 3V3INT 3V3EN.Q2.UP"
- board text removed: "0V 24V O0.7 O0.6 O0.5 O0.4 O0.3 O0.2 O0.1 Q0.0"
- board text removed: "0V 24V O1.7 O1.6 O1.5 O1.4 O1.3 O1.2 O1.1 Q1.0"
- board text removed: "24V/5V"
- board text removed: "Base Board V2.6 M36 2023-07-30"
- board text removed: "Experimental Study C.Niesen, Königswinter, Germany, CC BY-NC-SA 2023"
- board text removed: "FFC/PFS Base Board V2.6 M36 2023-07-30"
- board text removed: "O0.0 O0.1 O0.2 O0.3 O0.4 O0.5 O0.6 O0.7 24V 0V"
- board text removed: "O1.0 O1.1 O1.2 O1.3 O1.4 O1.5 O1.6 O1.7 24V 0V"
- board text removed: "RESET MISO MOSI SPISCK SPICSIO GNDD 3V3INT"
