File: PLC/V4_KiCad_PCB/OP.kicad_pcb (KiCad board)
At the start: 2 copper layers, 208 x 80 mm, 306 parts, among them J1 MSTBVA-2.5-10-5.08, J10 01x03_fem, J11 01x02_fem, J12 01x15_fem, J13 01x03_fem, J14 01x15_fem, J15 01x04_fem, J16 MSTBVA-2.5-10-5.08, J17 MSTBVA-2.5-10-5.08, J2 MSTBVA-2.5-10-5.08, J25 01x05_fem, J27 Lötauge, J28 GND_CAN opt an J33, J3 PFS 2x4, J33 opt. GND_XXX, J37 Lötauge, J4 01x08_fem, J40 Extention, J41 Lötauge, J42 Lötauge, J43 Flachstecker, J44 Lötauge, J45 Lötauge, J46 Lötauge, J47 Lötauge, J48 Lötauge, J5 01x04_fem, J51 Lötauge, J52 Lötauge, J6 DIN-5, J61 Lötauge, J62 Lötauge, J7 DIN-5, J8 02x02_fem, J9 Ub 0V PE, P1 1,0K lin, P2 1,0K lin, Q1 IRLML 2244, SW1 SW_DIP_x02, SW2 SW_DIP_x02, SW3 SW_DIP_x02, U1 LTV-844, U10 ADM2483xRW, U2 LTV-844, U3 LTV-844, U36 MCP3204, U39 ADuM1401xRW, U4 LTV-844, U42 LM4040 AIM3-2.5, U43 LM4040 AIM3-2.5, U47 ADM-809Z, U48 ADM-803L, U49 74AHC1G32, U5 MCP23S17, U50 NE555DRG4, U6 ISO1050, U7 Teensy4.0, U8 ISO1050, U9 25LC512

Commit message: Final version V2.9 M41
Cold start issues solved.
Parts:
- removed D50: 3V0, Diodes_SMD:D_MiniMELF
- removed U48: ADM-803L, TO_SOT_Packages_SMD:SOT-23
- added J36: 01x01_fem, Connector_PinSocket_2.54mm:PinSocket_1x01_P2.54mm_Vertical, B.Cu at (105.5, 58.4)
- C1: value 100µ 6V3 -> Siehe Text
- R126: value 2k7 -> 220
- U49: value 74AHC1G32 -> SN74LV1T32DBVR
- moved C71 1.53 mm to (164.6, 60.4), turned to 90 degrees
- moved R163 1.17 mm to (86.9, 75.4)
- moved R165 0.86 mm to (86.9, 77.5)
- moved C99 0.39 mm to (243.1, 76.6)
- moved R126 0.32 mm to (161.9, 63.5)
- moved C70 0.25 mm to (161.7, 61.3)
- moved R171 0.06 mm to (162.8, 55.0)
Connections:
- R126 pad 2: 5V_CPU_IN -> Net-(J36-Pad1)
Routing:
- net Net-(J36-Pad1): track 0.00 -> 118.9 mm, vias 0 -> 2
- net /3V3_INT: track 370.6 -> 419.9 mm, vias 16 -> 15
- net Net-(C48-Pad1): track 46.1 -> 14.8 mm, vias 10 -> 32
- net GNDD: track 692.1 -> 714.0 mm, vias 161 -> 166
- net /~RESET: track 152.0 -> 133.9 mm
- net 5V_CPU_IN: track 119.6 -> 103.8 mm
- net /GND_CAN_BUS: track 141.0 -> 151.8 mm, vias 8 -> 9
- net /PE: track 1068.7 -> 1072.8 mm
- net /~SW_MODE_2: track 30.8 -> 28.0 mm
- net /RS485_B: track 59.9 -> 57.5 mm
- net GNDA: track 67.8 -> 68.6 mm
- net Net-(R163-Pad2): track 2.78 -> 1.97 mm
- net /GND_RS485_BUS: track 65.9 -> 66.6 mm
- net /CAN2TX: track 145.4 -> 145.9 mm
- added copper zone on In1.Cu, net /GND_CAN_BUS
- added copper zone on In2.Cu, net /GND_CAN_BUS
- added copper zone on In1.Cu, net /GND_RS485_BUS
- added copper zone on In2.Cu, net /GND_RS485_BUS
- added copper zone on In1.Cu, net /PE
- added copper zone on In2.Cu, net /PE
- added copper zone on In1.Cu, net /U0V
- added copper zone on In2.Cu, net /U0V
- added copper zone on In1.Cu, net GNDA
- added copper zone on In2.Cu, net GNDA
- added copper zone on In1.Cu, net GNDD
- added copper zone on In2.Cu, net GNDD
- added copper zone on In1.Cu, net Net-(C48-Pad1)
- added copper zone on In2.Cu, net Net-(C48-Pad1)
- added copper zone on In1.Cu, net Net-(C59-Pad1)
- added copper zone on In2.Cu, net Net-(C59-Pad1)
Other:
- copper layers 2 -> 4
- board text added: "*"
- board text added: "3V3INT GNDD 3V3 ADDA GNDA"
- board text added: "4Layer PCB"
- board text added: "FFC CPU Board V2.9 M41 2024-06-09"
- board text added: "GNDD CPU 5V 3V3"
- board text added: "In1"
- board text added: "In2"
- board text added: "J3: BAT3V6 ~SWMODE2 ~RESET ~SWMODE1 GND n.c."
- board text removed: "3V3INTF GNDD 3V3 ADDA GNDA"
- board text removed: "BAT 3V ~RESET ~SWMODE1 ~SWMODE2"
- board text removed: "GNDD CPU 5V"
- board text removed: "J3: BAT 3V ~RESET ~SWMODE1 ~SWMODE2"
- board text removed: "J3: GNDD O O GNDD O O GNDD O O GNDD O O"
- board text removed: "O O GNDD O O GNDD O O GNDD O O GNDD"
- board text removed: "PFS CPU Board V2.8 M40 2024-05-27"
