File: PLC/V5_KiCad_PCB/OP.kicad_pcb (KiCad board)
At the start: 4 copper layers, 208 x 80 mm, 335 parts, among them J1 MSTBVA-2.5-10-5.08, J10 01x03_fem, J11 01x02_fem, J12 01x15_fem, J13 01x03_fem, J14 01x15_fem, J15 01x04_fem, J16 MSTBVA-2.5-10-5.08, J17 MSTBVA-2.5-10-5.08, J2 MSTBVA-2.5-10-5.08, J25 01x05_fem, J27 Lötauge, J28 GND_CAN, J3 Conn_02x04_Odd_Even, J36 01x01_fem, J37 Lötauge, J4 01x08_fem, J40 Extention, J41 Lötauge, J42 Lötauge, J43 Flachstecker, J44 Lötauge, J45 Lötauge, J46 Lötauge, J5 01x04_fem, J51 Lötauge, J52 Lötauge, J6 DIN-5, J61 Lötauge, J62 Lötauge, J7 DIN-5, J8 02x02_fem, J9 Ub 0V PE, P1 1,0K lin, P2 1,0K lin, Q1 IRLML 2244, SW1 SW_DIP_x02, SW2 SW_DIP_x02, SW3 GDS0204, SW4 OnOff, SW5 Prog, U1 LTV-844, U10 ADM2483xRW, U2 LTV-844, U3 LTV-844, U36 MCP3204, U39 ADuM1401xRW, U4 LTV-844, U42 LM4040 AIM3-2.5, U43 LM4040 AIM3-2.5, U47 ADM-809Z, U48 TPS3431, U49 SN74LV1T32, U5 MCP23S17, U50 NE555DRG4, U52 S-80929CNMC, U53 BD7LS04G-C, U54 BD7LS04G-C, U6 ISO1050, U7 Teensy4.0, U8 ISO1050, U9 25LC512

Commit message: Final V5 Upload
Uploading final Version May 2026 V5
PCB, Partslist, Sheets.
Doku outstanding
Parts:
- added R50: 220, myLib9:R_0805, B.Cu at (170.7, 81.3)
- added U40: ADM-803S, Package_TO_SOT_SMD:SOT-23, B.Cu at (170.7, 78.3)
- C106: value 3µ3 10V -> 2µ2; footprint Capacitor_Tantalum_SMD:CP_EIA-3216-18_Kemet-A -> Capacitor_SMD:C_1206_3216Metric
- C2: moved to B.Cu
- moved C2 15.6 mm to (157.5, 83.6), turned to 0 degrees
- moved R150 0.38 mm to (175.9, 77.1)
Connections:
- D34 pad 1: /CAN1H -> /CAN2H
- D34 pad 2: /CAN1L -> /CAN2L
- D35 pad 1: /CAN2L -> /CAN1L
- D35 pad 2: /CAN2H -> /CAN1H
- J6 pad 1: /CAN1L -> /CAN2L
- J6 pad 3: /CAN2L -> /CAN1L
- J6 pad 4: /CAN1H -> /CAN2H
- J6 pad 5: /CAN2H -> /CAN1H
- J7 pad 3: /CAN2L -> /CAN1L
- J7 pad 5: /CAN2H -> /CAN1H
- SW1 pad 3: /CAN1H -> /CAN2H
- SW1 pad 4: /CAN1L -> /CAN2L
- SW2 pad 3: /CAN2L -> /CAN1L
- SW2 pad 4: /CAN2H -> /CAN1H
- U6 pad 2: /CAN1RX -> /CAN2RX
- U6 pad 3: /CAN1TX -> /CAN2TX
- U6 pad 6: /CAN1L -> /CAN2L
- U6 pad 7: /CAN1H -> /CAN2H
- U8 pad 2: /CAN2RX -> /CAN1RX
- U8 pad 3: /CAN2TX -> /CAN1TX
- U8 pad 6: /CAN2L -> /CAN1L
- U8 pad 7: /CAN2H -> /CAN1H
Routing:
- net /CAN2L: track 80.7 -> 57.5 mm, vias 1 -> 0
- net /CAN1L: track 57.5 -> 80.7 mm, vias 0 -> 1
- net /CAN2H: track 74.8 -> 52.2 mm, vias 1 -> 0
- net /CAN1H: track 52.2 -> 74.8 mm, vias 0 -> 1
- net 3V3: track 132.4 -> 152.3 mm, vias 4 -> 6
- net /CAN2TX: track 145.8 -> 164.5 mm, vias 1 -> 2
- net GNDD: track 1280.4 -> 1261.9 mm, vias 130 -> 125
- net /CAN2RX: track 144.0 -> 162.1 mm, vias 1 -> 2
- net /~{RESET}: track 135.4 -> 146.9 mm, vias 3 -> 4
- net /CAN1RX: track 169.8 -> 159.3 mm
- net /CAN1TX: track 170.2 -> 162.5 mm
- net /TR-U50: track 21.1 -> 28.4 mm, vias 1 -> 2
- net /3V3_INT: track 424.4 -> 420.2 mm, vias 14 -> 13
- net /3V3EN_Q2_UP: track 37.2 -> 37.9 mm
Other:
- board text added: "+"
- board text added: "-"
- board text added: "Experimental Study PS4 1xx-MMx substitution CPU Board C.Niesen,Königswinter,Germany, (RS485-ORG) CC BY-NC-SA 2020-2026"
- board text added: "PFS CPU Board V3.2 M43 2026-05-17"
- board text added: "WDdelay ms 5,7*C106/nF 2µ2~12sec"
- board text added: "myT40-PLC V5"
- board text added: "myT40-PLC with Teensy 4.0 V5"
- board text removed: "Experimental Study PS4 1xx-MMx substitution CPU Board C.Niesen,Königswinter,Germany, (RS485-ORG % UP M42) CC BY-NC-SA 2020-2025"
- board text removed: "PFS CPU Board V3.1 M43 2025-08-14"
- board text removed: "WDdelay ms 5,7*C106/nF 3µ3~18sec"
- board text removed: "myT40-PLC"
- board text removed: "myT40-PLC with Teensy 4.0"
