File: PLC/V5_KiCad_PCB/UP.kicad_pcb (KiCad board)
At the start: 2 copper layers, 208 x 80 mm, 254 parts, among them J18 01x03_Male, J19 01x08_Male, J20 01x02_Male, J21 02x02_Male, J22 opt. Connector, J23 opt. Connector, J24 01x05_Male, J26 01x04_Male, J29 Lötauge, J30 Lötauge, J31 Lötauge, J32 Lötauge, J34 01x01_Male, J35 Lötauge, J38 Lötauge, J39 Lötauge, J49 01x15 Male zu OP, J50 01x15 Male zu OP, J53 Lötauge, J54 Lötauge, J55 Lötauge, J56 Lötauge, J57 Lötauge, J58 Lötauge, J59 Lötauge, J60 Lötauge, J63 Lötauge, J64 Lötauge, J65 Lötauge, J66 Flachstecker, Q2 IRLML 2244, U11 2S7WA_2405_S3RP, U12 2S7WA_2405_S3RP, U13 LT1086 3.3, U14 MCP23S17, U15 LTV-844, U16 LTV-844, U17 LTV-844, U18 LTV-844, U19 BSP-452, U20 BSP-452, U21 BSP-452, U22 BSP-452, U23 BSP-452, U24 BSP-452, U25 BSP-452, U26 BSP-452, U27 BSP-452, U28 BSP-452, U29 BSP-452, U30 BSP-452, U31 BSP-452, U32 BSP-452, U33 BSP-452, U34 BSP-452, U35 ADuM1401xRW, U37 LT1086 3.3, U38 MCP4922, U40 ADM-803S, U41 LT 1078, U44 2S7WB_2415S3RP, U45 ADR03ARZ, U46 LCN78_05-1.0, U51 SN74LV1T08

Commit message: Final V5 Upload
Uploading final Version May 2026 V5
PCB, Partslist, Sheets.
Doku outstanding
Parts:
- removed R50: 220, myLib9:R_0805
- removed U40: ADM-803S, Package_TO_SOT_SMD:SOT-23
Routing:
- net /~{RESET}: track 19.9 -> 20.6 mm
Other:
- board text added: "Base Board V3.2 M43 2026-05-17"
- board text added: "Experimental Study: PS4-1xx-MMx BaseBoard C.Niesen, Königswinter, Germany, CC BY-NC-SA 2020-2026"
- board text added: "FFC/PFS Base Board V3.2 M43 2026-05-17"
- board text added: "myT40-PLC with Teensy 4.0 V5"
- board text removed: "Base Board V3.1 M43 2025-08-14"
- board text removed: "Experimental Study: PS4-1xx-MMx BaseBoard C.Niesen, Königswinter, Germany, CC BY-NC-SA 2020-2025"
- board text removed: "FFC/PFS Base Board V3.1 M43 2025-08-14"
- board text removed: "myT40-PLC with Teensy 4.0"
