File: myT40-PLC/V5_KiCad_PCB/OP.kicad_pcb (KiCad board)
At the start: 4 copper layers, 208 x 80 mm, 337 parts, among them J1 MSTBVA-2.5-10-5.08, J10 01x03_fem, J11 01x02_fem, J12 01x15_fem, J13 01x03_fem, J14 01x15_fem, J15 01x04_fem, J16 MSTBVA-2.5-10-5.08, J17 MSTBVA-2.5-10-5.08, J2 MSTBVA-2.5-10-5.08, J25 01x05_fem, J27 Lötauge, J28 GND_CAN, J3 Conn_02x04_Odd_Even, J36 01x01_fem, J37 Lötauge, J4 01x08_fem, J40 Extention, J41 Lötauge, J42 Lötauge, J43 Flachstecker, J44 Lötauge, J45 Lötauge, J46 Lötauge, J5 01x04_fem, J51 Lötauge, J52 Lötauge, J6 DIN-5, J61 Lötauge, J62 Lötauge, J7 DIN-5, J8 02x02_fem, J9 Ub 0V PE, P1 1,0K lin, P2 1,0K lin, Q1 IRLML 2244, SW1 SW_DIP_x02, SW2 SW_DIP_x02, SW3 GDS0204, SW4 OnOff, SW5 Prog, U1 LTV-844, U10 ADM2483xRW, U2 LTV-844, U3 LTV-844, U36 MCP3204, U39 ADuM1401xRW, U4 LTV-844, U40 ADM-803S, U42 LM4040 AIM3-2.5, U43 LM4040 AIM3-2.5, U47 ADM-809Z, U48 TPS3431, U49 SN74LV1T32, U5 MCP23S17, U50 NE555DRG4, U52 S-80929CNMC, U53 BD7LS04G-C, U54 BD7LS04G-C, U6 ISO1050, U7 Teensy4.0, U8 ISO1050, U9 25LC512

Commit message: myT40-PLC V5 ready to production
myT40-PLC Rev3.3 M44 V5
Documentation reduced to V5
Parts:
- removed D52: BZY55B3V0, Diode_SMD:D_0805_2012Metric
- removed R173: 330, myLib9:R_0805
- added C108: 100n, Capacitor_SMD:C_1206_3216Metric, B.Cu at (241.7, 88.9)
- added J33: 01x03_fem, Connector_PinSocket_2.54mm:PinSocket_1x03_P2.54mm_Vertical, B.Cu at (98.9, 91.3)
- added RV4: 46VAC, Resistor_SMD:R_1210_3225Metric, F.Cu at (76.0, 106.1)
- added RV5: 46VAC, Resistor_SMD:R_1210_3225Metric, B.Cu at (82.8, 50.9)
- added RV6: 46VAC, Resistor_SMD:R_1210_3225Metric, F.Cu at (88.4, 68.1)
- added U55: FM25V10, Package_SO:SOIC-8_5.3x6.2mm_P1.27mm, F.Cu at (242.1, 88.9)
- C24, L2: moved to B.Cu
- C8: footprint myLib9:C_1206_HandSoldering -> Capacitor_SMD:C_0805_2012Metric
- C9: footprint myLib9:C_1206_HandSoldering -> Capacitor_SMD:C_1206_3216Metric
- J25: value 01x05_fem -> 01x02_fem; footprint Connector_PinSocket_2.54mm:PinSocket_1x05_P2.54mm_Vertical -> Connector_PinSocket_2.54mm:PinSocket_1x02_P2.54mm_Vertical
- J3: value Conn_02x04_Odd_Even -> 02x04
- J36: value 01x01_fem -> 01x03_fem; footprint Connector_PinSocket_2.54mm:PinSocket_1x01_P2.54mm_Vertical -> Connector_PinSocket_2.54mm:PinSocket_1x03_P2.54mm_Vertical
- J8: value 02x02_fem -> 01x02_fem; footprint Connector_PinSocket_2.54mm:PinSocket_2x02_P2.54mm_Vertical -> Connector_PinSocket_2.54mm:PinSocket_1x02_P2.54mm_Vertical
- JP6: value GND-DEF-J7 -> GND-DEF.J7; footprint Connector_PinHeader_2.00mm:PinHeader_1x03_P2.00mm_Vertical -> Connector_PinHeader_2.54mm:PinHeader_1x03_P2.54mm_Vertical
- R133: footprint Resistor_SMD:R_1206_3216Metric -> Resistor_SMD:R_0805_2012Metric
- R174: footprint Resistor_SMD:R_0805_2012Metric -> Resistor_SMD:R_1206_3216Metric
- R62: footprint myLib9:R_1206_HandSoldering -> Resistor_SMD:R_1206_3216Metric; moved to B.Cu
- moved C24 11.6 mm to (109.6, 109.1), turned to -90 degrees
- moved TP5 11.0 mm to (100.6, 68.8)
- moved R152 10.0 mm to (185.3, 79.5), turned to 90 degrees
- moved C104 8.50 mm to (185.1, 46.6)
- moved C105 8.50 mm to (177.8, 46.6)
- moved SW4 8.18 mm to (185.2, 43.9)
- moved SW5 7.85 mm to (177.8, 43.9)
- moved C78 5.67 mm to (172.1, 43.2)
- moved J36 5.24 mm to (106.8, 53.3), turned to 180 degrees
- moved C9 5.08 mm to (242.1, 85.1), turned to 0 degrees
- moved J51 2.84 mm to (102.1, 83.8), turned to 90 degrees
- moved R62 2.54 mm to (242.1, 92.7), turned to 180 degrees
- moved C8 2.53 mm to (101.6, 79.9)
- moved D36 2.44 mm to (85.5, 83.0)
- moved R131 1.53 mm to (112.2, 97.1)
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Connections:
- net /PE renamed PE
- net Net-(JP1-C) renamed /~{WP}
- net Net-(U9-MISO) renamed /MISO_0
- J36 pad 1: 3V3 -> GNDD
- J8 pad 1: /GND_CAN_BUS -> /Ub_CAN_BUS
- J8 pad 2: GNDD -> /GND_CAN_BUS
Routing:
- net PE: track 1056.4 -> 933.7 mm, vias 59 -> 61
- net GNDD: track 1261.9 -> 1221.7 mm, vias 125 -> 118
- net (no net): track 0.00 -> 40.0 mm
- net /LED2: track 197.8 -> 160.5 mm, vias 2 -> 1
- net /LED3: track 189.9 -> 152.9 mm, vias 2 -> 1
- net /LED1: track 227.6 -> 192.1 mm, vias 5 -> 2
- net GNDA: track 68.4 -> 93.0 mm, vias 38 -> 37
- net /Ub_CAN_BUS: track 72.9 -> 54.5 mm
- net /GND_RS485_BUS: track 60.7 -> 44.8 mm, vias 5 -> 6
- net /SPISCK: track 202.9 -> 187.1 mm
- net /3V3_INT: track 420.2 -> 406.4 mm
- net /CAN2TX: track 164.5 -> 152.8 mm, vias 2 -> 1
- net Net-(Q1-D): track 29.0 -> 40.3 mm, vias 1 -> 3
- net /CAN2RX: track 162.1 -> 153.2 mm, vias 2 -> 1
- net /~{WP}: track 12.0 -> 20.7 mm
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- added copper zone on In1.Cu, net /GND_RS485_BUS
- removed copper zone on In1.Cu, net /U0V
- removed copper zone on In2.Cu, net /U0V
Other:
- board text added: "*3"
- board text added: "/"
- board text added: "3V3_ADDA GNDA"
- board text added: "5V CANBUS GND"
- board text added: "<-JP6"
- board text added: "ADCDAC: U11 GNDA U10 U1 U0 Q0.4 Q0.3 Q0.2 Q0.1 Q0.0"
- board text added: "BAT3V6 GND ~{RESET} GND ~{SWMODE1} GND ~{SWMODE2} GND"
- board text added: "CAN1RX"
- board text added: "CAN1TX"
- board text added: "D44 D46"
- board text added: "D45 D47"
- board text added: "J3: GGND BAT3V6 GGND ~{RESET} GGND ~{SWMODE1} GGND ~{SWMODE2}"
- board text added: "PFS CPU Board V3.3 M44 2026-07-25"
- board text added: "X"
- board text removed: "3V3INT GNDD 3V3 ADDA GNDA"
- board text removed: ">JP6<"
- board text removed: "BAT3V6 GND ~{RESET} GND ~{SWMODE1} GND ~{SWMODE2} GND J3"
- board text removed: "J3: BAT3V6 ~{SWMODE2} ~{RESET} ~{SWMODE1} GND 1 N.C."
- board text removed: "J8 GND CANBUS 5V"
- board text removed: "PFS CPU Board V3.2 M43 2026-05-17"
