File: myT40-PLC/V5_KiCad_PCB/UP.kicad_pcb (KiCad board)
At the start: 2 copper layers, 208 x 80 mm, 252 parts, among them J18 01x03_Male, J19 01x08_Male, J20 01x02_Male, J21 02x02_Male, J22 opt. Connector, J23 opt. Connector, J24 01x05_Male, J26 01x04_Male, J29 Lötauge, J30 Lötauge, J31 Lötauge, J32 Lötauge, J34 01x01_Male, J35 Lötauge, J38 Lötauge, J39 Lötauge, J49 01x15 Male zu OP, J50 01x15 Male zu OP, J53 Lötauge, J54 Lötauge, J55 Lötauge, J56 Lötauge, J57 Lötauge, J58 Lötauge, J59 Lötauge, J60 Lötauge, J63 Lötauge, J64 Lötauge, J65 Lötauge, J66 Flachstecker, Q2 IRLML 2244, U11 2S7WA_2405_S3RP, U12 2S7WA_2405_S3RP, U13 LT1086 3.3, U14 MCP23S17, U15 LTV-844, U16 LTV-844, U17 LTV-844, U18 LTV-844, U19 BSP-452, U20 BSP-452, U21 BSP-452, U22 BSP-452, U23 BSP-452, U24 BSP-452, U25 BSP-452, U26 BSP-452, U27 BSP-452, U28 BSP-452, U29 BSP-452, U30 BSP-452, U31 BSP-452, U32 BSP-452, U33 BSP-452, U34 BSP-452, U35 ADuM1401xRW, U37 LT1086 3.3, U38 MCP4922, U41 LT 1078, U44 2S7WB_2415S3RP, U45 ADR03ARZ, U46 LCN78_05-1.0, U51 SN74LV1T08

Commit message: myT40-PLC V5 ready to production
myT40-PLC Rev3.3 M44 V5
Documentation reduced to V5
Parts:
- removed D106, D107, D108, D109, D110, D111, D112, D113, D114, D115, D116, D117, D118, D119, D120, D121: 1N4448W7F DII, myLib9:Diode_DO213AB-MELF_SOD123
- removed R102, R103, R104, R105, R106, R107, R108, R109, R110, R111, R112, R113, R114, R115, R116, R117: 7k5, Resistor_SMD:R_1206_3216Metric
- added J47: 01x03_Male, Connector_PinHeader_2.54mm:PinHeader_1x03_P2.54mm_Vertical, F.Cu at (98.9, 91.3)
- C98: footprint Capacitor_SMD:C_1206_3216Metric -> Capacitor_SMD:C_0805_2012Metric
- J21: value 02x02_Male -> 01x02_Male; footprint Connector_PinHeader_2.54mm:PinHeader_2x02_P2.54mm_Vertical -> Connector_PinHeader_2.54mm:PinHeader_1x02_P2.54mm_Vertical
- J24: value 01x05_Male -> 01x02_Male; footprint Connector_PinHeader_2.54mm:PinHeader_1x05_P2.54mm_Vertical -> Connector_PinHeader_2.54mm:PinHeader_1x02_P2.54mm_Vertical
- J29: value Lötauge -> DAC 3pol J29-J31
- J34: value 01x01_Male -> 01x03_Male; footprint Connector_PinHeader_2.54mm:PinHeader_1x01_P2.54mm_Vertical -> Connector_PinHeader_2.54mm:PinHeader_1x03_P2.54mm_Vertical
- R141: moved to B.Cu
- moved R136 17.4 mm to (231.3, 77.7), turned to -90 degrees
- moved R134 17.3 mm to (244.0, 77.7), turned to -90 degrees
- moved R138 16.9 mm to (218.6, 77.7), turned to -90 degrees
- moved R144 16.5 mm to (148.2, 78.0), turned to -90 degrees
- moved R146 16.5 mm to (135.5, 78.0), turned to -90 degrees
- moved R148 16.4 mm to (122.8, 78.0), turned to -90 degrees
- moved R140 16.3 mm to (205.9, 77.7), turned to -90 degrees
- moved R142 16.3 mm to (160.9, 78.0), turned to -90 degrees
- moved R135 7.73 mm to (236.6, 65.4), turned to -90 degrees
- moved R141 6.36 mm to (198.4, 65.4), turned to -90 degrees
- moved R137 5.66 mm to (223.9, 65.4), turned to -90 degrees
- moved J34 5.24 mm to (106.8, 53.3)
- moved R147 4.94 mm to (128.7, 65.3), turned to -90 degrees
- moved C17 4.90 mm to (99.2, 54.3), turned to -90 degrees
- moved R149 4.78 mm to (116.7, 66.3)
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Connections:
- D54 pad 1: Net-(D106-A) -> Net-(D54-K)
- D55 pad 1: Net-(D107-A) -> Net-(D55-K)
- D56 pad 1: Net-(D108-A) -> Net-(D56-K)
- D57 pad 1: Net-(D109-A) -> Net-(D57-K)
- D58 pad 1: Net-(D110-A) -> Net-(D58-K)
- D59 pad 1: Net-(D111-A) -> Net-(D59-K)
- D60 pad 1: Net-(D112-A) -> Net-(D60-K)
- D61 pad 1: Net-(D113-A) -> Net-(D61-K)
- D62 pad 1: Net-(D114-A) -> Net-(D62-K)
- D63 pad 1: Net-(D115-A) -> Net-(D63-K)
- D64 pad 1: Net-(D116-A) -> Net-(D64-K)
- D65 pad 1: Net-(D117-A) -> Net-(D65-K)
- D66 pad 1: Net-(D118-A) -> Net-(D66-K)
- D67 pad 1: Net-(D119-A) -> Net-(D67-K)
- D68 pad 1: Net-(D120-A) -> Net-(D68-K)
- D69 pad 1: Net-(D121-A) -> Net-(D69-K)
- J21 pad 1: /GND_CAN_BUS -> /Ub_CAN_BUS
- J21 pad 2: GNDD -> /GND_CAN_BUS
- J34 pad 1: 3V3 -> GNDD
- R134 pad 2: Net-(U19-IN) -> Net-(D61-K)
- R135 pad 2: Net-(U20-IN) -> Net-(D60-K)
- R136 pad 2: Net-(U21-IN) -> Net-(D59-K)
- R137 pad 2: Net-(U22-IN) -> Net-(D58-K)
- R138 pad 2: Net-(U23-IN) -> Net-(D57-K)
- R139 pad 2: Net-(U24-IN) -> Net-(D56-K)
- R140 pad 2: Net-(U25-IN) -> Net-(D55-K)
- R141 pad 2: Net-(U26-IN) -> Net-(D54-K)
- R142 pad 2: Net-(U27-IN) -> Net-(D69-K)
- R143 pad 2: Net-(U28-IN) -> Net-(D68-K)
- R144 pad 2: Net-(U29-IN) -> Net-(D67-K)
- R145 pad 2: Net-(U30-IN) -> Net-(D66-K)
- R146 pad 2: Net-(U31-IN) -> Net-(D65-K)
- R147 pad 2: Net-(U32-IN) -> Net-(D64-K)
- R148 pad 2: Net-(U33-IN) -> Net-(D63-K)
- R149 pad 2: Net-(U34-IN) -> Net-(D62-K)
- U15 pad 11: Net-(U21-IN) -> Net-(D59-A)
- U15 pad 13: Net-(U20-IN) -> Net-(D60-A)
- U15 pad 15: Net-(U19-IN) -> Net-(D61-A)
- U15 pad 9: Net-(U22-IN) -> Net-(D58-A)
- U16 pad 11: Net-(U25-IN) -> Net-(D55-A)
- U16 pad 13: Net-(U24-IN) -> Net-(D56-A)
- U16 pad 15: Net-(U23-IN) -> Net-(D57-A)
- U16 pad 9: Net-(U26-IN) -> Net-(D54-A)
- U17 pad 11: Net-(U29-IN) -> Net-(D67-A)
- U17 pad 13: Net-(U28-IN) -> Net-(D68-A)
- U17 pad 15: Net-(U27-IN) -> Net-(D69-A)
- U17 pad 9: Net-(U30-IN) -> Net-(D66-A)
- U18 pad 11: Net-(U33-IN) -> Net-(D63-A)
- U18 pad 13: Net-(U32-IN) -> Net-(D64-A)
- U18 pad 15: Net-(U31-IN) -> Net-(D65-A)
- U18 pad 9: Net-(U34-IN) -> Net-(D62-A)
- U19 pad 3: Net-(U19-IN) -> Net-(D61-K)
- U20 pad 3: Net-(U20-IN) -> Net-(D60-K)
- U21 pad 3: Net-(U21-IN) -> Net-(D59-K)
- U22 pad 3: Net-(U22-IN) -> Net-(D58-K)
- U23 pad 3: Net-(U23-IN) -> Net-(D57-K)
- U24 pad 3: Net-(U24-IN) -> Net-(D56-K)
- U25 pad 3: Net-(U25-IN) -> Net-(D55-K)
- U26 pad 3: Net-(U26-IN) -> Net-(D54-K)
- U27 pad 3: Net-(U27-IN) -> Net-(D69-K)
- U28 pad 3: Net-(U28-IN) -> Net-(D68-K)
- U29 pad 3: Net-(U29-IN) -> Net-(D67-K)
- U30 pad 3: Net-(U30-IN) -> Net-(D66-K)
- U31 pad 3: Net-(U31-IN) -> Net-(D65-K)
- U32 pad 3: Net-(U32-IN) -> Net-(D64-K)
- U33 pad 3: Net-(U33-IN) -> Net-(D63-K)
- U34 pad 3: Net-(U34-IN) -> Net-(D62-K)
Routing:
- net /PE: track 198.4 -> 423.1 mm, vias 100 -> 104
- net /GNDPWR_Out_0: track 342.2 -> 263.2 mm, vias 13 -> 8
- net /GNDPWR_Out_1: track 317.2 -> 258.2 mm, vias 13 -> 10
- net Net-(D60-A): track 0.00 -> 56.3 mm
- net Net-(D61-A): track 0.00 -> 54.5 mm
- net Net-(D58-A): track 0.00 -> 53.3 mm
- net Net-(D59-A): track 0.00 -> 51.6 mm
- net Net-(D56-A): track 0.00 -> 50.2 mm
- net Net-(D65-A): track 0.00 -> 50.0 mm
- net Net-(D67-A): track 0.00 -> 49.9 mm
- net Net-(D69-A): track 0.00 -> 49.9 mm
- net Net-(D57-A): track 0.00 -> 49.6 mm
- net Net-(D68-A): track 0.00 -> 49.5 mm
- net Net-(D62-A): track 0.00 -> 49.3 mm
- net Net-(D66-A): track 0.00 -> 49.1 mm
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Other:
- board text added: "5V CAN"
- board text added: "Base Board V3.3 M44 2026-07-25"
- board text added: "CAN BUS GND 5V CAN"
- board text added: "FFC/PFS Base Board V3.3 M44 2026-07-25"
- board text added: "GND CANBUS"
- board text removed: "Base Board V3.2 M43 2026-05-17"
- board text removed: "CAN BUS GNDC 5V"
- board text removed: "FFC/PFS Base Board V3.2 M43 2026-05-17"
